File: Schematics/Tagger.sch (KiCad schematic (older format))
At the start: 40 parts, among them J3 I2C_ToReceiverModules, J4 ToSerialBT, SW1 SW_Push, SW2 SW_Push, T2 BC237, T3 Q_NMOS_DGS, T4 BC237, T5 BC237, T6 BC237, T7 BC237, T8 BC237, T9 BC237, U1 PCF8574A, U2 MCP6001R

Commit message: New Version of Tagger/Receiver Schematics and PCBs
Parts:
- removed D4, D5, D6: LED_ARGB, LEDs:LED_D5.0mm-4, symbol LED_ARGB
- removed D7, D8, D9: MuzzleFireLED, LEDs:LED_D5.0mm-4, symbol LED_ARGB
- removed R7, R8: R, Resistors_THT:R_Axial_DIN0207_L6.3mm_D2.5mm_P2.54mm_Vertical, symbol R
- removed T8, T9: BC237, TO_SOT_Packages_THT:TO-92_Molded_Narrow, symbol BC237
- removed U2: MCP6001R, Housings_DIP:DIP-8_W7.62mm, symbol MCP6001R
- added D? (x6): LED_CRGB, symbol LED_CRGB
- added D? (x2): D, symbol D
- added J? (x2): Conn_01x02_Female, symbol Conn_01x02_Female
- added J?: Conn_01x07_Female, symbol Conn_01x07_Female
- added R?: 150R, Resistors_THT:R_Axial_DIN0207_L6.3mm_D2.5mm_P2.54mm_Vertical, symbol R
- added R? (x2): R, symbol R
- LD1: symbol Laserdiode_1A3C -> Laserdiode_1A3C-RESCUE-Tagger
- R1: value R -> 22k
- R12: value R -> 150R
- R13: value R -> 1k5
- R14: value R -> 1k
- R2: value R -> 33k
- renumbered T7 to T1
Connections:
- net +5V: now also T4.1 (C), T5.1 (C), T6.1 (C)
- net GND: now also D?.1 (K), D?.1 (K), D?.1 (K), D?.1 (K), D?.1 (K), D?.1 (K); no longer R10.2, R11.2, R9.2, T4.1 (C), T5.1 (C), T6.1 (C)
- net at R12.2: now also D?.2 (RA), D?.2 (RA), D?.2 (RA), R?.2
- net at R13.2: now also D?.3 (GA), D?.3 (GA), D?.3 (GA)
- net at R14.2: now also D?.4 (BA), D?.4 (BA), D?.4 (BA)
- net at D2.2 (A): now also R?.1; no longer A1.10 ((PCINT23/AIN1)PD7)
- net at D1.2 (A): now also R?.1; no longer A1.9 ((PCINT22/OC0A/AIN0)PD6)
- net at T3.3 (S): now also R10.1, R11.1, R9.1
- net at T3.2 (G): now also A1.10 ((PCINT23/AIN1)PD7); no longer A1.11 (PCINT0/CLK0/ICP1)PB0)
- net at R12.1, T4.3 (E): now also R?.1
- net at R5.2, R6.2: now also T1.2 (B); no longer D3.2 (A)
- net at T1.1 (C): now also A1.7 ((PCINT20/XCK/T0)PD4)
- net at A1.8 ((PCINT21/OC0B/T1)PD5): now also R?.2
- net at R6.1: now also D?.1 (K)
- net at R5.1: now also D?.1 (K); no longer T1.3 (E)
- net at T2.2 (B): now also A1.11 (PCINT0/CLK0/ICP1)PB0); no longer A1.12 ((PCINT1/OC1A)PB1)
- net at A1.13 ((PCINT2/OC1B/~SS~)PB2): now also D?.2 (A); no longer T1.2 (B)
- net at A1.14 ((PCINT3/OC2A/MOSI)PB3): now also J?.1 (Pin_1)
- net at A1.15 ((PCINT4/MISO)PB4): now also J?.2 (Pin_2)
- net at A1.16 ((PCINT5/SCK/LED)PB5): now also J?.1 (Pin_1)
- net +3V3: now reaches A1.17 (+3.3V)
- net +3V3: now also J?.2 (Pin_2)
- net VAA: now reaches A1.18 (AREF)
- net VAA: now also J?.3 (Pin_3)
- net at A1.19 ((PCINT8/ADC0)PC0): now also J?.4 (Pin_4)
- net at A1.20 ((PCINT9/ADC1)PC1): now also J?.5 (Pin_5)
- net at A1.21 ((PCINT10/ADC2)PC2): now also J?.6 (Pin_6)
- net at A1.22 ((PCINT11/ADC3)PC3): now also J?.7 (Pin_7)
- net at A1.25 (ADC6): now also J?.1 (Pin_1)
- net at A1.26 (ADC7): now also J?.2 (Pin_2)
- new net: D?.4 (BA), D?.4 (BA), D?.4 (BA), R9.2
- new net: D?.3 (GA), D?.3 (GA), D?.3 (GA), R10.2
- new net: D?.2 (RA), D?.2 (RA), D?.2 (RA), R11.2
- new net: D3.2 (A), T1.3 (E)
- new net: A1.12 ((PCINT1/OC1A)PB1), D?.2 (A)
- new net: A1.9 ((PCINT22/OC0A/AIN0)PD6), R?.2
Other:
- moved on the sheet: D1, D2, D3, R10, R11, R5, R6, R9, T1, T3, T4, T5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
